File: JONAHS HACKPAD/JONAHS HACKPAD/PCB Pro Files/PRO/PRO.kicad_pcb (KiCad board)
At the start: 2 copper layers, 61.9 x 82.3 mm, 42 parts, among them SW2 SW_Push, SW3 SW_Push, SW4 SW_Push, SW5 SW_Push, U1 MOUDLE-SEEEDUINO-XIAO, U2 OLED_0.91_128x32

Commit message: update stuff
Parts:
- removed C1, C10, C11, C12, C13, C14, C15, C2, C3, C4, C5, C6, C7, C8, C9: 100nF, Capacitor_SMD:C_0805_2012Metric
- removed C16: 10uF, Capacitor_SMD:C_0805_2012Metric
- removed R1: 470R, Resistor_SMD:R_0805_2012Metric
Connections:
- RE1 pad A: Net-(U1-PA7_A8_D8_SCK) -> Net-(D6-DIN)
- U1 pad 8: Net-(U1-PA7_A8_D8_SCK) -> Net-(D6-DIN)
- U1 pad 9: Net-(U1-PA7_A8_D8_SCK) -> Net-(D6-DIN)
Routing:
- net GND: track 353.1 -> 246.8 mm, vias 2 -> 3
- net Net-(D10-VDD): track 253.8 -> 189.8 mm, vias 5 -> 2
- net Net-(U1-PA7_A8_D8_SCK): track 46.1 -> 0.00 mm, vias 1 -> 0
- net Net-(D6-DIN): track 39.9 -> 65.2 mm, vias 1 -> 2
- net Net-(D8-DOUT): track 46.3 -> 61.5 mm
- net Net-(D17-K): track 21.5 -> 30.1 mm, vias 1 -> 2
- net Net-(U1-PA5_A9_D9_MISO): track 52.3 -> 47.1 mm, vias 1 -> 0
- net Net-(D10-DIN): track 29.2 -> 33.9 mm
- net Net-(D1-K): track 46.4 -> 42.5 mm
- net Net-(D2-A): track 31.7 -> 28.6 mm
- net Net-(D5-K): track 86.4 -> 84.9 mm
- net Net-(D6-DOUT): track 28.2 -> 26.8 mm
- net Net-(D7-DOUT): track 34.6 -> 33.3 mm
- net Net-(D4-K): track 67.9 -> 69.0 mm
- net Net-(U1-PA8_A4_D4_SDA): track 43.4 -> 42.6 mm, vias 0 -> 1
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